Commit message: Added Hardware and Navigation files

File: medibot_description/urdf/materials.xacro (robot description, xacro)
@@ -5,8 +5,11 @@
 </material>
 <material name="steel_satin">
-  <color rgba="0.6274509803921569 0.6274509803921569 0.6274509803921569 1.0"/>
+  <color rgba="0.4 0.4 0.4 1.0"/>
 </material>
 <material name="plastic_translucent_glossy_gray">
-  <color rgba="0.7019607843137254 0.7019607843137254 0.7019607843137254 0.0"/>
+  <color rgba="0.1 0.1 0.1 1.0"/>
+</material>
+<material name="blue">
+  <color rgba="0.1 0.1 0.7 1.0"/>
 </material>
 </robot>

File: medibot_description/urdf/medibot.xacro (robot description, xacro)
@@ -35,5 +35,5 @@
       <mesh filename="package://medibot_description/meshes/lidar_1.stl" scale="0.001 0.001 0.001"/>
     </geometry>
-    <material name="steel_satin"/>
+    <material name="blue"/>
   </visual>
   <collision>

Commit message: Updated new URDF

File: medibot_description/urdf/materials.xacro (robot description, xacro)
@@ -4,6 +4,6 @@
   <color rgba="0.700 0.700 0.700 1.000"/>
 </material>
-<material name="steel_satin">
-  <color rgba="0.4 0.4 0.4 1.0"/>
+<material name="black">
+  <color rgba="0.2 0.2 0.2 1.0"/>
 </material>
 <material name="plastic_translucent_glossy_gray">

File: medibot_description/urdf/medibot.xacro (robot description, xacro)
@@ -6,7 +6,7 @@
 <link name="base_link">
   <inertial>
-    <origin xyz="0.12348117476989938 0.030658625276350104 0.04780371902134241" rpy="0 0 0"/>
-    <mass value="10.161748166428781"/>
-    <inertia ixx="0.152266" iyy="0.143569" izz="0.265149" ixy="-0.032066" iyz="0.017667" ixz="0.00919"/>
+    <origin xyz="0.04581707300319793 0.0010479310706408762 0.07330638052099143" rpy="0 0 0"/>
+    <mass value="6.358114447165492"/>
+    <inertia ixx="0.037035" iyy="0.038312" izz="0.055341" ixy="-0.000504" iyz="-1.1e-05" ixz="-0.00176"/>
   </inertial>
   <visual>
@@ -15,5 +15,5 @@
       <mesh filename="package://medibot_description/meshes/base_link.stl" scale="0.001 0.001 0.001"/>
     </geometry>
-    <material name="steel_satin"/>
+    <material name="black"/>
   </visual>
   <collision>
@@ -24,32 +24,12 @@
   </collision>
 </link>
-<link name="lidar_1">
+<link name="l_wheel_1">
   <inertial>
-    <origin xyz="-0.268067 0.0 -0.1408" rpy="0 0 0"/>
-    <mass value="0.0"/>
-    <inertia ixx="0.0" iyy="0.0" izz="0.0" ixy="0.0" iyz="0.0" ixz="0.0"/>
+    <origin xyz="2.1103228532710293e-07 0.0037429225188824466 7.237266341775239e-15" rpy="0 0 0"/>
+    <mass value="0.8943597759780031"/>
+    <inertia ixx="0.000733" iyy="0.001393" izz="0.000733" ixy="0.0" iyz="-0.0" ixz="0.0"/>
   </inertial>
   <visual>
-    <origin xyz="-0.268067 -0.0 -0.1408" rpy="0 0 0"/>
-    <geometry>
-      <mesh filename="package://medibot_description/meshes/lidar_1.stl" scale="0.001 0.001 0.001"/>
-    </geometry>
-    <material name="blue"/>
-  </visual>
-  <collision>
-    <origin xyz="-0.268067 -0.0 -0.1408" rpy="0 0 0"/>
-    <geometry>
-      <mesh filename="package://medibot_description/meshes/lidar_1.stl" scale="0.001 0.001 0.001"/>
-    </geometry>
-  </collision>
-</link>
-<link name="l_wheel_1">
-  <inertial>
-    <origin xyz="-8.806132971057051e-15 0.003742975244019703 8.167078124898808e-15" rpy="0 0 0"/>
-    <mass value="0.8943597759780031"/>
-    <inertia ixx="0.000733" iyy="0.001393" izz="0.000733" ixy="-0.0" iyz="-0.0" ixz="0.0"/>
-  </inertial>
-  <visual>
-    <origin xyz="0.0 -0.1282 -0.05" rpy="0 0 0"/>
+    <origin xyz="-0.0 -0.1292 -0.05" rpy="0 0 0"/>
     <geometry>
       <mesh filename="package://medibot_description/meshes/l_wheel_1.stl" scale="0.001 0.001 0.001"/>
@@ -58,5 +38,5 @@
   </visual>
   <collision>
-    <origin xyz="0.0 -0.1282 -0.05" rpy="0 0 0"/>
+    <origin xyz="-0.0 -0.1292 -0.05" rpy="0 0 0"/>
     <geometry>
       <mesh filename="package://medibot_description/meshes/l_wheel_1.stl" scale="0.001 0.001 0.001"/>
@@ -66,10 +46,10 @@
 <link name="r_wheel_1">
   <inertial>
-    <origin xyz="4.220585108133287e-15 -0.0037429752440196196 4.378442053365461e-15" rpy="0 0 0"/>
+    <origin xyz="2.1103229032957658e-07 -0.003743027969156404 5.044575868140555e-15" rpy="0 0 0"/>
     <mass value="0.8943597759780031"/>
     <inertia ixx="0.000733" iyy="0.001393" izz="0.000733" ixy="0.0" iyz="0.0" ixz="0.0"/>
   </inertial>
   <visual>
-    <origin xyz="0.0 0.1282 -0.05" rpy="0 0 0"/>
+    <origin xyz="-0.0 0.1292 -0.05" rpy="0 0 0"/>
     <geometry>
       <mesh filename="package://medibot_description/meshes/r_wheel_1.stl" scale="0.001 0.001 0.001"/>
@@ -78,5 +58,5 @@
   </visual>
   <collision>
-    <origin xyz="0.0 0.1282 -0.05" rpy="0 0 0"/>
+    <origin xyz="-0.0 0.1292 -0.05" rpy="0 0 0"/>
     <geometry>
       <mesh filename="package://medibot_description/meshes/r_wheel_1.stl" scale="0.001 0.001 0.001"/>
@@ -84,20 +64,40 @@
   </collision>
 </link>
+<link name="lidar_1">
+  <inertial>
+    <origin xyz="-0.155 -8.8e-05 -0.1428" rpy="0 0 0"/>
+    <mass value="0.0"/>
+    <inertia ixx="0.0" iyy="0.0" izz="0.0" ixy="0.0" iyz="0.0" ixz="0.0"/>
+  </inertial>
+  <visual>
+    <origin xyz="-0.155 -8.8e-05 -0.1428" rpy="0 0 0"/>
+    <geometry>
+      <mesh filename="package://medibot_description/meshes/lidar_1.stl" scale="0.001 0.001 0.001"/>
+    </geometry>
+    <material name="blue"/>
+  </visual>
+  <collision>
+    <origin xyz="-0.155 -8.8e-05 -0.1428" rpy="0 0 0"/>
+    <geometry>
+      <mesh filename="package://medibot_description/meshes/lidar_1.stl" scale="0.001 0.001 0.001"/>
+    </geometry>
+  </collision>
+</link>
+<joint name="base2left" type="continuous">
+  <origin xyz="0.0 0.1292 0.05" rpy="0 0 0"/>
+  <parent link="base_link"/>
+  <child link="l_wheel_1"/>
+  <axis xyz="0.0 1.0 0.0"/>
+</joint>
+<joint name="base2right" type="continuous">
+  <origin xyz="0.0 -0.1292 0.05" rpy="0 0 0"/>
+  <parent link="base_link"/>
+  <child link="r_wheel_1"/>
+  <axis xyz="0.0 1.0 0.0"/>
+</joint>
 <joint name="base2lidar" type="fixed">
-  <origin xyz="0.268067 0.0 0.1408" rpy="0 0 0"/>
+  <origin xyz="0.155 8.8e-05 0.1428" rpy="0 0 0"/>
   <parent link="base_link"/>
   <child link="lidar_1"/>
 </joint>
-<joint name="base2left" type="continuous">
-  <origin xyz="0.0 0.1282 0.05" rpy="0 0 0"/>
-  <parent link="base_link"/>
-  <child link="l_wheel_1"/>
-  <axis xyz="0.0 1.0 -0.0"/>
-</joint>
-<joint name="base2right" type="continuous">
-  <origin xyz="0.0 -0.1282 0.05" rpy="0 0 0"/>
-  <parent link="base_link"/>
-  <child link="r_wheel_1"/>
-  <axis xyz="-0.0 -1.0 0.0"/>
-</joint>
 </robot>
